Commit message: turn gravity off

File: urdf/general_aruco.urdf.xacro (robot description, xacro)
@@ -4,5 +4,5 @@
     <xacro:arg name="aruco_id" default="0"/>
     <xacro:arg name="aruco_name" default="DICT_4X4_50_id0"/>
-    <xacro:arg name="aruco_l" default="0.2"/>
+    <xacro:arg name="aruco_l" default="0.5"/>
     <xacro:arg name="white_border" default="0.1"/>
     <xacro:include filename="$(find aruco_description)/urdf/general_aruco.xacro"/>

File: urdf/general_aruco.xacro (robot description, xacro)
@@ -21,10 +21,10 @@
         <inertia ixx="0.0741666666667" ixy="0.0" ixz="0.0" iyy="0.0585416666667" iyz="0.0" izz="0.0260416666667"/>
       </inertial>
-      <collision>
+      <!-- <collision>
         <origin xyz="0 0 0" rpy="0 0 0"/>
         <geometry>
           <box size="${aruco_l + 2*white_border * aruco_l} ${aruco_l + 2*white_border * aruco_l} ${0.01 * aruco_l/0.09}"/>
         </geometry>
-      </collision>
+      </collision> -->
       <visual>
         <origin xyz="0 0 0" rpy="0 0 0"/>
@@ -42,9 +42,10 @@
     </link>
     <gazebo reference="${aruco_name}_link_0">
-      <kp>100000.0</kp>
-      <kd>100000.0</kd>
+      <kp>0.0</kp>
+      <kd>0.0</kd>
       <mu1>0.1</mu1>
       <mu2>0.1</mu2>
       <fdir1>1 0 0</fdir1>
+      <turnGravityOff>1</turnGravityOff>
     </gazebo>
   </xacro:macro>
